Commit message: Change EEF to tool0

File: m710ic70_7axis.urdf (robot description, URDF)
Before this commit: robot m710ic70, 9 links, 8 joints
Links:
- added link tool0
Joints:
- added joint link_6-tool0: type fixed, parent flange, child tool0, origin xyz=0 0 0 rpy=3.14159 -1.570795 0

Commit message: change joint name of e1

File: m710ic70_7axis.urdf (robot description, URDF)
Before this commit: robot m710ic70_7axis, 10 links, 9 joints
Joints:
- removed joint e_1
- added joint joint_e1: type prismatic, parent base_link, child link_e1, origin xyz=0 0 0 rpy=0 0 0, axis 1 0 0, limit lower=0.0 upper=10.0 effort=0 velocity=0.5

Commit message: change j3 limit
* j3 is coupling with j2
* see https://robodk.com/forum/Thread-Fanuc-M710-iC-45M-J2-J3-coupling

File: m710ic70_7axis.urdf (robot description, URDF)
Before this commit: robot m710ic70_7axis, 10 links, 9 joints
Joints:
- joint joint_3: limit lower=-2.7925 upper=4.8869 effort=0 velocity=3.0543 -> lower=-1.405 upper=3.5779 effort=0 velocity=3.0543
